File: Elettronica/No-Brim Scheme.kicad_pcb (KiCad board)
At the start: 2 copper layers, 38 parts, among them J1 Conn_01x09, J10 Motor 24v, J2 24V, J3 Elettrovalve_1M1, J4 Elettrovalve_2M1, J5 Elettrovalve_3M1, J6 Elettrovalve_4M1, J7 Elettrovalve_1M2, J8 Elettrovalve_2M2, J9 Elettrovalve_3M2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

Commit message: PCB completato da revisionare(16/6)
Parts:
- J1: value Conn_01x09 -> Conn_01x10; footprint Connector_PinSocket_2.54mm:PinSocket_1x09_P2.54mm_Vertical -> Connector_PinSocket_2.54mm:PinSocket_1x10_P2.54mm_Vertical
- moved K1 86.7 mm to (21.3, 84.6), turned to 90 degrees
- moved J6 84.0 mm to (55.9, 81.3)
- moved J3 21.0 mm to (55.9, 33.5)
- moved J4 21.0 mm to (55.9, 50.0)
- moved J7 21.0 mm to (55.9, 41.7)
- moved J5 20.9 mm to (55.9, 65.3)
- moved J8 20.9 mm to (55.9, 57.1)
- moved J9 20.9 mm to (55.9, 73.2)
- moved J10 20.3 mm to (46.7, 82.8), turned to 270 degrees
- moved J2 6.86 mm to (46.2, 35.1)
Routing:
- net +24V: track 0.51 -> 135.1 mm
- net Net-(D4-Pad2): track 4.96 -> 32.3 mm, vias 0 -> 1
- net Net-(D3-Pad2): track 3.48 -> 24.3 mm, vias 0 -> 1
- net Net-(D9-Pad2): track 5.59 -> 25.6 mm
- net Net-(D7-Pad2): track 3.01 -> 22.7 mm, vias 0 -> 1
- net Net-(D1-Pad2): track 5.06 -> 23.9 mm
- net Net-(D2-Pad2): track 5.06 -> 23.4 mm, vias 0 -> 1
- net Net-(D8-Pad2): track 2.76 -> 17.0 mm
- net Net-(D6-Pad2): track 3.01 -> 16.5 mm, vias 0 -> 1
- net Net-(D5-Pad2): track 2.50 -> 15.2 mm, vias 0 -> 1
- net Net-(K1-Pad7): track 0.00 -> 7.62 mm
- net GND: track 187.5 -> 191.5 mm
- net Motor_230v: track 21.0 -> 20.1 mm
Other:
- board text added: "No-Brim Project 2020"
