File: Elettronica/No-Brim Scheme.sch (KiCad schematic (older format))
At the start: 27 parts, among them J1 Conn_01x06, J2 Elettrovalve_1, J3 Motor 24v, J4 24V, J5 230V, J6 Elettrovalve_2, J7 Motor 230V, J8 Elettrovalve_3, J9 Elettrovalve_4, Q1 IRLML0030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

Commit message: Modifiche allo schema e pcb recuperato(16/6)
Parts:
- removed D4: D, symbol Device:D
- removed J1: Conn_01x06, symbol Connector_Generic:Conn_01x06
- removed J5: 230V, symbol Connector_Generic:Conn_01x02
- removed J7: Motor 230V, symbol Connector_Generic:Conn_01x02
- removed Q4: IRF7799L2, Package_DirectFET:DirectFET_L8, symbol Transistor_FET:IRF7799L2
- removed R4: R, symbol Device:R
- added D5, D6, D7, D9: D, Diode_SMD:D_2010_5025Metric_Pad1.52x2.65mm_HandSolder, symbol No-Brim-Scheme-rescue:D-Device
- added J1: Conn_01x09, Connector_PinSocket_2.54mm:PinSocket_1x09_P2.54mm_Vertical, symbol No-Brim-Scheme-rescue:Conn_01x09-Connector_Generic
- added J7: Elettrovalve_1M2, Connector_PinSocket_2.54mm:PinSocket_1x02_P2.54mm_Vertical, symbol No-Brim-Scheme-rescue:Conn_01x02-Connector_Generic
- added J8: Elettrovalve_2M2, Connector_PinSocket_2.54mm:PinSocket_1x02_P2.54mm_Vertical, symbol No-Brim-Scheme-rescue:Conn_01x02-Connector_Generic
- added J9: Elettrovalve_3M2, Connector_PinSocket_2.54mm:PinSocket_1x02_P2.54mm_Vertical, symbol No-Brim-Scheme-rescue:Conn_01x02-Connector_Generic
- added K1: DIPxx-1Cxx-51x, Relay_THT:Relay_StandexMeder_DIP_LowProfile, symbol No-Brim-Scheme-rescue:DIPxx-1Cxx-51x-Relay
- added Q5, Q6, Q7, Q9: IRLML0030, Package_TO_SOT_SMD:SOT-23, symbol No-Brim-Scheme-rescue:IRLML0030-Transistor_FET
- added R5, R6, R7, R9: R, Resistor_SMD:R_1206_3216Metric_Pad1.42x1.75mm_HandSolder, symbol No-Brim-Scheme-rescue:R-Device
- D1: footprint (none) -> Diode_SMD:D_2010_5025Metric_Pad1.52x2.65mm_HandSolder; symbol Device:D -> No-Brim-Scheme-rescue:D-Device
- D2: renamed from D3; footprint (none) -> Diode_SMD:D_2010_5025Metric_Pad1.52x2.65mm_HandSolder; symbol Device:D -> No-Brim-Scheme-rescue:D-Device
- D3: renamed from D5; footprint (none) -> Diode_SMD:D_2010_5025Metric_Pad1.52x2.65mm_HandSolder; symbol Device:D -> No-Brim-Scheme-rescue:D-Device
- D4: renamed from D6; footprint (none) -> Diode_SMD:D_2010_5025Metric_Pad1.52x2.65mm_HandSolder; symbol Device:D -> No-Brim-Scheme-rescue:D-Device
- D8: renamed from D2; footprint (none) -> Diode_SMD:D_2010_5025Metric_Pad1.52x2.65mm_HandSolder; symbol Device:D -> No-Brim-Scheme-rescue:D-Device
- J10: renamed from J3; footprint (none) -> Connector_PinSocket_2.54mm:PinSocket_1x02_P2.54mm_Vertical; symbol Connector_Generic:Conn_01x02 -> No-Brim-Scheme-rescue:Conn_01x02-Connector_Generic
- J2: renamed from J4; footprint (none) -> Connector_PinSocket_2.00mm:PinSocket_1x02_P2.00mm_Vertical; symbol Connector_Generic:Conn_01x02 -> No-Brim-Scheme-rescue:Conn_01x02-Connector_Generic
- J3: renamed from J2; value Elettrovalve_1 -> Elettrovalve_1M1; footprint (none) -> Connector_PinSocket_2.54mm:PinSocket_1x02_P2.54mm_Vertical; symbol Connector_Generic:Conn_01x02 -> No-Brim-Scheme-rescue:Conn_01x02-Connector_Generic
- J4: renamed from J6; value Elettrovalve_2 -> Elettrovalve_2M1; footprint (none) -> Connector_PinSocket_2.54mm:PinSocket_1x02_P2.54mm_Vertical; symbol Connector_Generic:Conn_01x02 -> No-Brim-Scheme-rescue:Conn_01x02-Connector_Generic
- J5: renamed from J8; value Elettrovalve_3 -> Elettrovalve_3M1; footprint (none) -> Connector_PinSocket_2.54mm:PinSocket_1x02_P2.54mm_Vertical; symbol Connector_Generic:Conn_01x02 -> No-Brim-Scheme-rescue:Conn_01x02-Connector_Generic
- J6: renamed from J9; value Elettrovalve_4 -> Elettrovalve_4M1; footprint (none) -> Connector_PinSocket_2.54mm:PinSocket_1x02_P2.54mm_Vertical; symbol Connector_Generic:Conn_01x02 -> No-Brim-Scheme-rescue:Conn_01x02-Connector_Generic
- Q1: symbol Transistor_FET:IRLML0030 -> No-Brim-Scheme-rescue:IRLML0030-Transistor_FET
- Q2: renamed from Q3; symbol Transistor_FET:IRLML0030 -> No-Brim-Scheme-rescue:IRLML0030-Transistor_FET
- Q3: renamed from Q5; symbol Transistor_FET:IRLML0030 -> No-Brim-Scheme-rescue:IRLML0030-Transistor_FET
- Q4: renamed from Q6; symbol Transistor_FET:IRLML0030 -> No-Brim-Scheme-rescue:IRLML0030-Transistor_FET
- Q8: renamed from Q2; symbol Transistor_FET:IRLML0030 -> No-Brim-Scheme-rescue:IRLML0030-Transistor_FET
- R1: footprint (none) -> Resistor_SMD:R_1206_3216Metric_Pad1.42x1.75mm_HandSolder; symbol Device:R -> No-Brim-Scheme-rescue:R-Device
- R2: renamed from R3; footprint (none) -> Resistor_SMD:R_1206_3216Metric_Pad1.42x1.75mm_HandSolder; symbol Device:R -> No-Brim-Scheme-rescue:R-Device
- R3: renamed from R5; footprint (none) -> Resistor_SMD:R_1206_3216Metric_Pad1.42x1.75mm_HandSolder; symbol Device:R -> No-Brim-Scheme-rescue:R-Device
- R4: renamed from R6; footprint (none) -> Resistor_SMD:R_1206_3216Metric_Pad1.42x1.75mm_HandSolder; symbol Device:R -> No-Brim-Scheme-rescue:R-Device
- R8: renamed from R2; footprint (none) -> Resistor_SMD:R_1206_3216Metric_Pad1.42x1.75mm_HandSolder; symbol Device:R -> No-Brim-Scheme-rescue:R-Device
Connections:
- net labels added: 1M1_1, 1M1_2, 2M1_1, 2M1_2, 3M1_1, 3M1_2, 4M1_1
- net labels removed: Ev_1, Ev_2, Ev_3, Ev_4, LINE
- wire segments 93 -> 131

Commit message: PCB completato da revisionare(16/6)
Parts:
- removed J1: Conn_01x09, Connector_PinSocket_2.54mm:PinSocket_1x09_P2.54mm_Vertical, symbol No-Brim-Scheme-rescue:Conn_01x09-Connector_Generic
- added J1: Conn_01x10, Connector_PinSocket_2.54mm:PinSocket_1x10_P2.54mm_Vertical, symbol Connector_Generic:Conn_01x10
Connections:
- net 1M1_1: now also J1.1 (Pin_1)
- net 1M1_2: now also J1.2 (Pin_2)
- net 2M1_1: now also J1.3 (Pin_3)
- net 2M1_2: now also J1.4 (Pin_4)
- net 3M1_1: now also J1.5 (Pin_5)
- net 3M1_2: now also J1.6 (Pin_6)
- net 4M1_1: now also J1.7 (Pin_7)
- net GND: now also J1.10 (Pin_10)
- net Motor_230v: now also J1.9 (Pin_9)
- net Motor_24v: now also J1.8 (Pin_8)
Changed lines of the file:
@@
 encoding utf-8
 Sheet 1 1
-Title ""
-Date ""
+Title "No-Brim project"
+Date "2020-06-16"
 Rev ""
-Comp ""
-Comment1 ""
+Comp "AFP 2019-2020"
+Comment1 "Schema elettrico scheda per Arduino"
 Comment2 ""
 Comment3 ""
@@
 Text GLabel 3950 6600 0    50   Input ~ 0
 4M1_1
-$Comp
-L No-Brim-Scheme-rescue:Conn_01x09-Connector_Generic J1
-U 1 1 5EF873A9
+Wire Wire Line
+	3950 5450 3950 5550
+$Comp
+L Connector_Generic:Conn_01x10 J1
+U 1 1 5EE90DB9
 P 950 1400
-F 0 "J1" H 868 775 50  0000 C CNN
-F 1 "Conn_01x09" H 868 866 50  0000 C CNN
-F 2 "Connector_PinSocket_2.54mm:PinSocket_1x09_P2.54mm_Vertical" H 950 1400 50  0001 C CNN
+F 0 "J1" H 1030 1392 50  0000 L CNN
+F 1 "Conn_01x10" H 1030 1301 50  0000 L CNN
+F 2 "Connector_PinSocket_2.54mm:PinSocket_1x10_P2.54mm_Vertical" H 950 1400 50  0001 C CNN
 F 3 "~" H 950 1400 50  0001 C CNN
 	1    950  1400
 	-1   0    0    -1
 $EndComp
-Wire Wire Line
-	3950 5450 3950 5550
+$Comp
+L No-Brim-Scheme-rescue:GND-power #PWR0101
+U 1 1 5EE9BC2F
+P 1150 1900
+F 0 "#PWR0101" H 1150 1650 50  0001 C CNN
+F 1 "GND-power" H 1155 1727 50  0000 C CNN
+F 2 "" H 1150 1900 50  0001 C CNN
+F 3 "" H 1150 1900 50  0001 C CNN
+	1    1150 1900
+	1    0    0    -1
+$EndComp
 $EndSCHEMATC

Commit message: 25/6
Parts:
- D1, D2, D3, D4, D5, D6, D7, D8, D9: symbol No-Brim-Scheme-rescue:D-Device -> No-Brim-Scheme-rescue:D-Device-No-Brim-Scheme-rescue
- J1: symbol Connector_Generic:Conn_01x10 -> No-Brim-Scheme-rescue:Conn_01x10-Connector_Generic
- J10, J2, J3, J4, J5, J6, J7, J8, J9: symbol No-Brim-Scheme-rescue:Conn_01x02-Connector_Generic -> No-Brim-Scheme-rescue:Conn_01x02-Connector_Generic-No-Brim-Scheme-rescue
- K1: symbol No-Brim-Scheme-rescue:DIPxx-1Cxx-51x-Relay -> No-Brim-Scheme-rescue:DIPxx-1Cxx-51x-Relay-No-Brim-Scheme-rescue
- Q1, Q2, Q3, Q4, Q5, Q6, Q7, Q8, Q9: symbol No-Brim-Scheme-rescue:IRLML0030-Transistor_FET -> No-Brim-Scheme-rescue:IRLML0030-Transistor_FET-No-Brim-Scheme-rescue
- R1, R2, R3, R4, R5, R6, R7, R8, R9: symbol No-Brim-Scheme-rescue:R-Device -> No-Brim-Scheme-rescue:R-Device-No-Brim-Scheme-rescue
